File: Tenn/Tenn.kicad_sch (KiCad schematic)
At the start: 29 parts, among them J1 Conn_01x02_Socket, J12 Conn_01x04_Female, J13 Conn_01x03_Male, J14 Conn_01x03_Male, J15 Conn_01x03_Male, J16 Conn_01x02_Male, J17 Conn_01x02_Male, J18 Conn_01x30_Pin, SW2 SW_Push, SW3 SW_Push, SW4 SW_SPDT, U1 L7805, U2 DRV8871DDA, U3 DRV8871DDA

Commit message: Updates to newest version of the PCB Changes size of 47uF capacitor Adds guide text on the back side for easier undertanding of the connections Fixes issues of unconnected vias and tracks
Parts:
- C5, C6: footprint Capacitor_SMD:C_0805_2012Metric_Pad1.18x1.45mm_HandSolder -> Capacitor_SMD:C_1206_3216Metric_Pad1.33x1.80mm_HandSolder
Changed lines of the file:
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@@
 (kicad_sch
-	(version 20231120)
+	(version 20250114)
 	(generator "eeschema")
-	(generator_version "8.0")
+	(generator_version "9.0")
 	(paper "A4")
 	(title_block
 		(title "DenjuDivision_Tenn_Minisumo_Board")
 		(date "2024-03-31")
-		(rev "1.0")
+		(rev "2.2")
 		(company "DenjuDivision")
 		(comment 1 "Design by Tenkai Cruz")
 		(comment 2 "@tenn.bots")
 	)
+	(rectangle
+		(start 139.7 38.1)
+		(end 180.34 73.66)
+		(stroke
+			(width 0)
+			(type default)
+		)
+		(fill
+			(type none)
+		)
+	)
+	(text "Arduino Nano"
+		(exclude_from_sim no)
+		(at 140.97 78.74 0)
+		(effects
+			(font
+				(size 1.27 1.27)
+			)
+			(justify left bottom)
+		)
+	)
+	(text "Sensor Connectors"
+		(exclude_from_sim no)
+		(at 39.37 78.74 0)
+		(effects
+			(font
+				(size 1.27 1.27)
+			)
+			(justify left bottom)
+		)
+	)
+	(text "Screen"
+		(exclude_from_sim no)
+		(at 90.17 78.74 0)
+		(effects
+			(font
+				(size 1.27 1.27)
+			)
+			(justify left bottom)
+		)
+	)
+	(text "Servo"
+		(exclude_from_sim no)
+		(at 90.17 129.54 0)
+		(effects
+			(font
+				(size 1.27 1.27)
+			)
+			(justify left bottom)
+		)
+	)
+	(text "Select Buttons"
+		(exclude_from_sim no)
+		(at 140.97 40.64 0)
+		(effects
+			(font
+				(size 1.27 1.27)
+			)
+			(justify left bottom)
+		)
+	)
+	(text "Motor Drivers"
+		(exclude_from_sim no)
+		(at 203.708 78.359 0)
+		(effects
+			(font
+				(size 1.27 1.27)
+			)
+			(justify left bottom)
+		)
+	)
+	(text "Remote"
+		(exclude_from_sim no)
+		(at 90.17 104.14 0)
+		(effects
+			(font
+				(size 1.27 1.27)
+			)
+			(justify left bottom)
+		)
+	)
+	(text "Power Supply and Voltage Regulator\n\n"
+		(exclude_from_sim no)
+		(at 39.37 43.18 0)
+		(effects
+			(font
+				(size 1.27 1.27)
+			)
+			(justify left bottom)
+		)
+	)
+	(text "Voltage Testing Pins"
+		(exclude_from_sim no)
+		(at 90.17 154.94 0)
+		(effects
+			(font
+				(size 1.27 1.27)
+			)
+			(justify left bottom)
+		)
+	)
 	(junction
 		(at 148.59 58.42)
@@
 		)
 	)
-	(rectangle
-		(start 139.7 38.1)
-		(end 180.34 73.66)
-		(stroke
-			(width 0)
-			(type default)
-		)
-		(fill
-			(type none)
-		)
-	)
-	(text "Arduino Nano"
-		(exclude_from_sim no)
-		(at 140.97 78.74 0)
-		(effects
-			(font
-				(size 1.27 1.27)
-			)
-			(justify left bottom)
-		)
-	)
-	(text "Sensor Connectors"
-		(exclude_from_sim no)
-		(at 39.37 78.74 0)
-		(effects
-			(font
-				(size 1.27 1.27)
-			)
-			(justify left bottom)
-		)
-	)
-	(text "Screen"
-		(exclude_from_sim no)
-		(at 90.17 78.74 0)
-		(effects
-			(font
-				(size 1.27 1.27)
-			)
-			(justify left bottom)
-		)
-	)
-	(text "Servo"
-		(exclude_from_sim no)
-		(at 90.17 129.54 0)
-		(effects
-			(font
-				(size 1.27 1.27)
-			)
-			(justify left bottom)
-		)
-	)
-	(text "Select Buttons"
-		(exclude_from_sim no)
-		(at 140.97 40.64 0)
-		(effects
-			(font
-				(size 1.27 1.27)
-			)
-			(justify left bottom)
-		)
-	)
-	(text "Motor Drivers"
-		(exclude_from_sim no)
-		(at 203.708 78.359 0)
-		(effects
-			(font
-				(size 1.27 1.27)
-			)
-			(justify left bottom)
-		)
-	)
-	(text "Remote"
-		(exclude_from_sim no)
-		(at 90.17 104.14 0)
-		(effects
-			(font
-				(size 1.27 1.27)
-			)
-			(justify left bottom)
-		)
-	)
-	(text "Power Supply and Voltage Regulator\n\n"
-		(exclude_from_sim no)
-		(at 39.37 43.18 0)
-		(effects
-			(font
-				(size 1.27 1.27)
-			)
-			(justify left bottom)
-		)
-	)
-	(text "Voltage Testing Pins"
-		(exclude_from_sim no)
-		(at 90.17 154.94 0)
-		(effects
-			(font
-				(size 1.27 1.27)
-			)
-			(justify left bottom)
-		)
-	)
 	(global_label "Sens8"
 		(shape input)
@@
 			)
 		)
-		(property "Footprint" "Capacitor_SMD:C_0805_2012Metric_Pad1.18x1.45mm_HandSolder"
+		(property "Footprint" "Capacitor_SMD:C_1206_3216Metric_Pad1.33x1.80mm_HandSolder"
 			(at 244.8052 109.22 0)
 			(effects
@@
 			)
 		)
-		(property "Footprint" "Capacitor_SMD:C_0805_2012Metric_Pad1.18x1.45mm_HandSolder"
+		(property "Footprint" "Capacitor_SMD:C_1206_3216Metric_Pad1.33x1.80mm_HandSolder"
 			(at 244.8052 146.05 0)
 			(effects
@@
 		)
 	)
+	(embedded_fonts no)
 )
